Commit message: complete khr-3hv

File: urdf/khr_arm/khr-arm.xacro (robot description, xacro)
@@ -4,12 +4,12 @@
 <xacro:include filename="$(find sotuken2017)/urdf/urdf_gazebo.xacro"/>
   <property name="ef" value="1.37293"/>
-  <property name="vel" value="0.14"/>
+  <property name="vel" value="7.5"/>
   <property name="arm_xy" value="0.026"/>
   <property name="shoulder_z" value="0.036"/>
-  <property name="shoulder_mass" value="0.02975"/>
+  <property name="shoulder_mass" value="0.0625"/>
   <property name="upper_arm_z" value="0.082"/>
-  <property name="upper_arm_mass" value="0.02975"/>
+  <property name="upper_arm_mass" value="0.0625"/>
   <property name="lower_arm_z" value="0.056"/>
-  <property name="lower_arm_mass" value="0.051"/>
+  <property name="lower_arm_mass" value="0.025"/>
  <xacro:macro name="make_arm" params="parent LRarm ref arm_bool">
      <joint name="${parent}_to_${LRarm}shoulder" type="revolute">
@@ -27,5 +27,5 @@
                 <box size="${arm_xy} ${arm_xy} ${shoulder_z}"/>
             </geometry>
-            <xacro:set_color/>
+            <xacro:black/>
         </visual>
         <collision>
@@ -59,5 +59,5 @@
                 <box size="${arm_xy} ${arm_xy} ${upper_arm_z}"/>
             </geometry>
-            <xacro:set_color/>
+            <xacro:black/>
         </visual>
         <collision>
@@ -86,5 +86,5 @@
                 <box size="${arm_xy} ${arm_xy} ${lower_arm_z}"/>
             </geometry>
-            <xacro:set_color/>
+            <xacro:black/>
         </visual>
         <collision>

File: urdf/khr_body/khr-body.xacro (robot description, xacro)
@@ -4,13 +4,13 @@
 <xacro:include filename="$(find sotuken2017)/urdf/urdf_gazebo.xacro"/>
   <property name="ef" value="1.37293"/>
-  <property name="vel" value="0.14"/>
+  <property name="vel" value="7.5"/>
   <property name="body_x" value="0.129"/>
   <property name="body_y" value="0.105"/>
   <property name="body_z" value="0.062"/>
-  <property name="body_mass" value="0.3655"/>
+  <property name="body_mass" value="0.3"/>
   <property name="body_2_x" value="0.057"/>
   <property name="body_2_y" value="0.08"/>
   <property name="body_2_z" value="0.041"/>
-  <property name="body_2_mass" value="0.3655"/>
+  <property name="body_2_mass" value="0.2"/>
   <xacro:macro name="default_origin">
 	  <origin xyz="0 0 0" rpy="0 0 0"/>
@@ -23,5 +23,5 @@
           <box size="${body_x} ${body_y} ${body_z}"/>
         </geometry>
-        <xacro:set_color/>
+        <xacro:gray/>
       </visual>
       <collision>
@@ -50,5 +50,5 @@
           <box size="${body_2_x} ${body_2_y} ${body_2_z}"/>
         </geometry>
-        <xacro:set_color/>
+        <xacro:black/>
       </visual>
 	  <collision>

File: urdf/khr_head/khr-head.xacro (robot description, xacro)
@@ -5,9 +5,9 @@
 <xacro:include filename="$(find sotuken2017)/urdf/khr_body/khr-body.xacro"/>
   <property name="ef" value="1.37293"/>
-  <property name="vel" value="0.14"/>
+  <property name="vel" value="7.5"/>
   <property name="head_x" value="0.052"/>
   <property name="head_y" value="0.031"/>
   <property name="head_z" value="0.033"/>
-  <property name="head_mass" value="0.119"/>
+  <property name="head_mass" value="0.1"/>
    <xacro:macro name="make_head" params="parent">
      <joint name="${parent}_to_head" type="revolute">
@@ -25,5 +25,5 @@
         		<box size="${head_x} ${head_y} ${head_z}"/>
        		</geometry>
-       		<xacro:set_color/>
+       		<xacro:gray/>
        	</visual>
        	<collision>

File: urdf/khr_leg/khr-leg normal.xacro (robot description, xacro)
@@ -5,5 +5,5 @@
 <xacro:include filename="$(find sotuken2017)/urdf/sensor/khr-force_sensor normal.xacro"/>
 	<property name="ef" value="1.37293"/>
-    <property name="vel" value="0.14"/>
+    <property name="vel" value="7.5"/>
 	<property name="leg_xy" value="0.03"/>
 	<property name="hips_z" value="0.0039"/>
@@ -15,6 +15,8 @@
 	<property name="shin_z" value="0.047"/>
 	<property name="shin_mass" value="0.068"/>
+	<property name="hizakozo_xz" value="0.01"/>
+	<property name="hizakozo_mass" value="0.01"/>
 	<property name="ankle_z" value="0.02"/>
-	<property name="ankle_mass" value="0.068"/>
+	<property name="ankle_mass" value="0.058"/>
 	<property name="foot_x" value="0.122"/>
 	<property name="foot_y" value="0.078"/>
@@ -117,15 +119,42 @@
 				</inertial>
 		</link>
-		<joint name="${LRleg}knee_to_${LRleg}shin" type="revolute">
+		<joint name="${LRleg}knee_to_${LRleg}hizakozo" type="revolute">
 				<parent link="${LRleg}knee"/>
+				<child link="${LRleg}hizakozo"/>
+				<origin xyz="0 0 -0.078" rpy="0 0 0"/>
+				<axis xyz="0 1 0"/>
+				<dynamics damping="0.5"/>
+				<limit lower="-0.0" upper="${M_PI / 2}" effort="${ef}" velocity="${vel}"/>
+		</joint>
+		<link name="${LRleg}hizakozo">
+				<visual>
+						<origin xyz="${hizakozo_xz} 0 -0.016" rpy="0 0 0"/>
+						<geometry>
+								<box size="${hizakozo_xz} ${leg_xy} ${hizakozo_xz}"/>
+						</geometry>
+						<xacro:black/>
+				</visual>
+				<collision>
+						<origin xyz="${hizakozo_xz} 0 -0.016" rpy="0 0 0"/>
+						<geometry>
+								<box size="${hizakozo_xz} ${leg_xy} ${hizakozo_xz}"/>
+						</geometry>
+				</collision>
+				<inertial>
+						<origin xyz="${hizakozo_xz} 0 -0.016" rpy="0 0 0"/>
+						<xacro:box_inertial m="${hizakozo_mass}" d="${hizakozo_xz}" w="${leg_xy}" h="${hizakozo_xz}"/>
+				</inertial>
+		</link>
+		<joint name="${LRleg}hizakozo_to_${LRleg}shin" type="revolute">
+				<parent link="${LRleg}hizakozo"/>
 				<child link="${LRleg}shin"/>
-				<origin xyz="-0.0205 0 -0.0885" rpy="0 0 0"/>
-				<axis xyz="0 1 0"/>
-				<dynamics damping="0.5"/>
-				<limit lower="-0.0" upper="${M_PI * 5 / 6}" effort="${ef}" velocity="${vel}"/>
+				<origin xyz="0 0 -0.032" rpy="0 0 0"/>
+				<axis xyz="0 1 0"/>
+				<dynamics damping="0.5"/>
+				<limit lower="-0.0" upper="${M_PI / 2}" effort="${ef}" velocity="${vel}"/>
 		</joint>
 		<link name="${LRleg}shin">
 				<visual>
-						<origin xyz="0.0205 0 -0.024" rpy="0 0 0"/>
+						<origin xyz="0 0 -0.0235" rpy="0 0 0"/>
 						<geometry>
 								<box size="${leg_xy} ${leg_xy} ${shin_z}"/>
@@ -134,5 +163,5 @@
 				</visual>
 				<collision>
-						<origin xyz="0.0205 0 -0.024" rpy="0 0 0"/>
+						<origin xyz="0 0 -0.0235" rpy="0 0 0"/>
 						<geometry>
 								<box size="${leg_xy} ${leg_xy} ${shin_z}"/>
@@ -140,5 +169,5 @@
 				</collision>
 				<inertial>
-						<origin xyz="0.0205 0 -0.024" rpy="0 0 0"/>
+						<origin xyz="0 0 -0.0235" rpy="0 0 0"/>
 						<xacro:box_inertial m="${shin_mass}" d="${leg_xy}" w="${leg_xy}" h="${shin_z}"/>
 				</inertial>
@@ -147,5 +176,5 @@
 				<parent link="${LRleg}shin"/>
 				<child link="${LRleg}ankle"/>
-				<origin xyz="0.0205 0 -0.0319" rpy="0 0 0"/>
+				<origin xyz="0 0 -0.0319" rpy="0 0 0"/>
 				<axis xyz="0 1 0"/>
 				<dynamics damping="0.5"/>
@@ -154,5 +183,5 @@
 		<link name="${LRleg}ankle">
 				<visual>
-						<origin xyz="0 0 -0.037" rpy="0 0 0"/>
+						<origin xyz="0 0 -0.04" rpy="0 0 0"/>
 						<geometry>
 								<box size="${leg_xy} ${leg_xy} ${ankle_z}"/>
@@ -161,5 +190,5 @@
 				</visual>
 				<collision>
-						<origin xyz="0 0 -0.037" rpy="0 0 0"/>
+						<origin xyz="0 0 -0.04" rpy="0 0 0"/>
 						<geometry>
 								<box size="${leg_xy} ${leg_xy} ${ankle_z}"/>
@@ -167,5 +196,5 @@
 				</collision>
 				<inertial>
-						<origin xyz="0 0 -0.037" rpy="0 0 0"/>
+						<origin xyz="0 0 -0.04" rpy="0 0 0"/>
 						<xacro:box_inertial m="${ankle_mass}" d="${leg_xy}" w="${leg_xy}" h="${ankle_z}"/>
 				</inertial>
@@ -181,5 +210,5 @@
 		<link name="${LRleg}foot">
 				<visual>
-						<origin xyz="0 ${ref * leg_xy / 2} -0.0315" rpy="0 0 0"/>
+						<origin xyz="0 ${ref * leg_xy / 2} -0.0312" rpy="0 0 0"/>
 						<geometry>
 								<box size="${foot_x} ${foot_y} ${foot_z}"/>
@@ -188,5 +217,5 @@
 				</visual>
 				<collision>
-						<origin xyz="0 ${ref * leg_xy / 2} -0.0315" rpy="0 0 0"/>
+						<origin xyz="0 ${ref * leg_xy / 2} -0.0312" rpy="0 0 0"/>
 						<geometry>
 								<box size="${foot_x} ${foot_y} ${foot_z}"/>
@@ -194,5 +223,5 @@
 				</collision>
 				<inertial>
-						<origin xyz="0 ${ref * leg_xy / 2} -0.0315" rpy="0 0 0"/>
+						<origin xyz="0 ${ref * leg_xy / 2} -0.0312" rpy="0 0 0"/>
 						<xacro:box_inertial m="${foot_mass}" d="${foot_x}" w="${foot_y}" h="${foot_z}"/>
 				</inertial>
@@ -211,8 +240,10 @@
 				<origin xyz="-${foot_x / 2 -0.015}  ${(ref * leg_xy / 2) - (foot_y / 2 - 0.015)} -${0.0315 + foot_z / 2 + box_z / 2}" rpy="0 0 0" />
 		</xacro:make_fsensor>
-		<joint name="${LRleg}foot_to_${LRleg}foot2" type="fixed">
+		<joint name="${LRleg}foot_to_${LRleg}foot2" type="revolute">
 				<parent link="${LRleg}foot"/>
 				<child link="${LRleg}foot2"/>
 				<origin xyz="0 ${ref * leg_xy / 2} -${0.0315 + foot_z / 2 + foot_z / 10 + box_z}" rpy="0 0 0"/>
+				<axis xyz="0 0 1"/>
+				<limit lower="-0" upper="0" effort="0" velocity="0"/>
 		</joint>
 		<link name="${LRleg}foot2">
@@ -238,4 +269,5 @@
 		<xacro:gazebo_link_black ref="${LRleg}thigh"/>
 		<xacro:gazebo_link_black ref="${LRleg}knee"/>
+		<xacro:gazebo_link_black ref="${LRleg}hizakozo"/>
 		<xacro:gazebo_link_black ref="${LRleg}shin"/>
 		<xacro:gazebo_link_black ref="${LRleg}ankle"/>

File: urdf/khr_leg/khr-leg.xacro (robot description, xacro)
@@ -6,20 +6,26 @@
 <xacro:include filename="$(find sotuken2017)/urdf/sensor/sensor-gazebo.xacro"/>
 	<property name="ef" value="1.37293"/>
-    <property name="vel" value="0.14"/>
+    <property name="vel" value="7.5"/>
 	<property name="leg_xy" value="0.03"/>
 	<property name="hips_z" value="0.0039"/>
-	<property name="hips_mass" value="0.03944"/>
+	<property name="hips_mass" value="0.048"/>
 	<property name="thigh_z" value="0.026"/>
-	<property name="thigh_mass" value="0.03944"/>
+	<property name="thigh_mass" value="0.068"/>
 	<property name="knee_z" value="0.088"/>
-	<property name="knee_mass" value="0.11832"/>
+	<property name="knee_mass" value="0.118"/>
 	<property name="shin_z" value="0.047"/>
-	<property name="shin_mass" value="0.04692"/>
+	<property name="shin_mass" value="0.068"/>
+	<property name="hizakozo_xz" value="0.01"/>
+	<property name="hizakozo_mass" value="0.01"/>
 	<property name="ankle_z" value="0.02"/>
-	<property name="ankle_mass" value="0.04692"/>
+	<property name="ankle_mass" value="0.058"/>
 	<property name="foot_x" value="0.122"/>
 	<property name="foot_y" value="0.078"/>
 	<property name="foot_z" value="0.01"/>
-	<property name="foot_mass" value="0.02346"/>
+	<property name="foot_mass" value="0.03"/>
+	<property name="foot2_x" value="0.122"/>
+	<property name="foot2_y" value="0.078"/>
+	<property name="foot2_z" value="0.002"/>
+	<property name="foot2_mass" value="0.05"/>
 	<xacro:macro name="make_leg" params="parent LRleg ref leg_bool">
  		<joint name="${parent}_to_${LRleg}hips" type="revolute">
@@ -42,5 +48,5 @@
     							<box size="${leg_xy} ${leg_xy} ${hips_z}"/>
   						</geometry>
-  						<xacro:set_color/>
+  						<xacro:black/>
   				</visual>
   				<collision>
@@ -74,5 +80,5 @@
 								<box size="${leg_xy} ${leg_xy} ${thigh_z}"/>
 						</geometry>
-						<xacro:set_color/>
+						<xacro:black/>
 				</visual>
 				<collision>
@@ -101,5 +107,5 @@
 								<box size="${leg_xy} ${leg_xy} ${knee_z}"/>
 						</geometry>
-						<xacro:set_color/>
+						<xacro:black/>
 				</visual>
 				<collision>
@@ -114,22 +120,49 @@
 				</inertial>
 		</link>
-		<joint name="${LRleg}knee_to_${LRleg}shin" type="revolute">
+		<joint name="${LRleg}knee_to_${LRleg}hizakozo" type="revolute">
 				<parent link="${LRleg}knee"/>
+				<child link="${LRleg}hizakozo"/>
+				<origin xyz="0 0 -0.078" rpy="0 0 0"/>
+				<axis xyz="0 1 0"/>
+				<dynamics damping="0.5"/>
+				<limit lower="-0.0" upper="${M_PI / 2}" effort="${ef}" velocity="${vel}"/>
+		</joint>
+		<link name="${LRleg}hizakozo">
+				<visual>
+						<origin xyz="${hizakozo_xz} 0 -0.016" rpy="0 0 0"/>
+						<geometry>
+								<box size="${hizakozo_xz} ${leg_xy} ${hizakozo_xz}"/>
+						</geometry>
+						<xacro:black/>
+				</visual>
+				<collision>
+						<origin xyz="${hizakozo_xz} 0 -0.016" rpy="0 0 0"/>
+						<geometry>
+								<box size="${hizakozo_xz} ${leg_xy} ${hizakozo_xz}"/>
+						</geometry>
+				</collision>
+				<inertial>
+						<origin xyz="${hizakozo_xz} 0 -0.016" rpy="0 0 0"/>
+						<xacro:box_inertial m="${hizakozo_mass}" d="${hizakozo_xz}" w="${leg_xy}" h="${hizakozo_xz}"/>
+				</inertial>
+		</link>
+		<joint name="${LRleg}hizakozo_to_${LRleg}shin" type="revolute">
+				<parent link="${LRleg}hizakozo"/>
 				<child link="${LRleg}shin"/>
-				<origin xyz="-0.0205 0 -0.0885" rpy="0 0 0"/>
+				<origin xyz="0 0 -0.032" rpy="0 0 0"/>
 				<axis xyz="0 1 0"/>
 				<dynamics damping="0.5"/>
-				<limit lower="-0.0" upper="${M_PI * 5 / 6}" effort="${ef}" velocity="${vel}"/>
+				<limit lower="-0.0" upper="${M_PI / 2}" effort="${ef}" velocity="${vel}"/>
 		</joint>
 		<link name="${LRleg}shin">
 				<visual>
-						<origin xyz="0.0205 0 -0.024" rpy="0 0 0"/>
+						<origin xyz="0 0 -0.0235" rpy="0 0 0"/>
 						<geometry>
 								<box size="${leg_xy} ${leg_xy} ${shin_z}"/>
 						</geometry>
-						<xacro:set_color/>
-				</visual>
-				<collision>
-						<origin xyz="0.0205 0 -0.024" rpy="0 0 0"/>
+						<xacro:black/>
+				</visual>
+				<collision>
+						<origin xyz="0 0 -0.0235" rpy="0 0 0"/>
 						<geometry>
 								<box size="${leg_xy} ${leg_xy} ${shin_z}"/>
@@ -137,5 +170,5 @@
 				</collision>
 				<inertial>
-						<origin xyz="0.0205 0 -0.024" rpy="0 0 0"/>
+						<origin xyz="0 0 -0.0235" rpy="0 0 0"/>
 						<xacro:box_inertial m="${shin_mass}" d="${leg_xy}" w="${leg_xy}" h="${shin_z}"/>
 				</inertial>
@@ -144,5 +177,5 @@
 				<parent link="${LRleg}shin"/>
 				<child link="${LRleg}ankle"/>
-				<origin xyz="0.0205 0 -0.0319" rpy="0 0 0"/>
+				<origin xyz="0 0 -0.0319" rpy="0 0 0"/>
 				<axis xyz="0 1 0"/>
 				<dynamics damping="0.5"/>
@@ -151,12 +184,12 @@
 		<link name="${LRleg}ankle">
 				<visual>
-						<origin xyz="0 0 -0.037" rpy="0 0 0"/>
+						<origin xyz="0 0 -0.04" rpy="0 0 0"/>
 						<geometry>
 								<box size="${leg_xy} ${leg_xy} ${ankle_z}"/>
 						</geometry>
-						<xacro:set_color/>
-				</visual>
-				<collision>
-						<origin xyz="0 0 -0.037" rpy="0 0 0"/>
+						<xacro:black/>
+				</visual>
+				<collision>
+						<origin xyz="0 0 -0.04" rpy="0 0 0"/>
 						<geometry>
 								<box size="${leg_xy} ${leg_xy} ${ankle_z}"/>
@@ -164,5 +197,5 @@
 				</collision>
 				<inertial>
-						<origin xyz="0 0 -0.037" rpy="0 0 0"/>
+						<origin xyz="0 0 -0.04" rpy="0 0 0"/>
 						<xacro:box_inertial m="${ankle_mass}" d="${leg_xy}" w="${leg_xy}" h="${ankle_z}"/>
 				</inertial>
@@ -178,12 +211,12 @@
 		<link name="${LRleg}foot">
 				<visual>
-						<origin xyz="0 ${ref * leg_xy / 2} -0.0315" rpy="0 0 0"/>
+						<origin xyz="0 ${ref * leg_xy / 2} -0.0312" rpy="0 0 0"/>
 						<geometry>
 								<box size="${foot_x} ${foot_y} ${foot_z}"/>
 						</geometry>
-						<xacro:set_color/>
-				</visual>
-				<collision>
-						<origin xyz="0 ${ref * leg_xy / 2} -0.0315" rpy="0 0 0"/>
+						<xacro:black/>
+				</visual>
+				<collision>
+						<origin xyz="0 ${ref * leg_xy / 2} -0.0312" rpy="0 0 0"/>
 						<geometry>
 								<box size="${foot_x} ${foot_y} ${foot_z}"/>
@@ -191,6 +224,45 @@
 				</collision>
 				<inertial>
-						<origin xyz="0 ${ref * leg_xy / 2} -0.0315" rpy="0 0 0"/>
+						<origin xyz="0 ${ref * leg_xy / 2} -0.0312" rpy="0 0 0"/>
 						<xacro:box_inertial m="${foot_mass}" d="${foot_x}" w="${foot_y}" h="${foot_z}"/>
+				</inertial>
+		</link>
+		<!-- set force sensor -->
+		<xacro:make_fsensor parent="${LRleg}foot" LR="${LRleg}" num="1">
+				<origin xyz="${foot_x / 2 - 0.015}  ${(ref * leg_xy / 2) + (foot_y / 2 - 0.015)} -${0.0315 + foot_z / 2 + box_z / 2}" rpy="0 0 0" />
+		</xacro:make_fsensor>
+		<xacro:make_fsensor parent="${LRleg}foot" LR="${LRleg}" num="2">
+				<origin xyz="-${foot_x / 2 -0.015}  ${(ref * leg_xy / 2) + (foot_y / 2 - 0.015)} -${0.0315 + foot_z / 2 + box_z / 2}" rpy="0 0 0" />
+		</xacro:make_fsensor>
+		<xacro:make_fsensor parent="${LRleg}foot" LR="${LRleg}" num="3">
+				<origin xyz="${foot_x / 2 -0.015}  ${(ref * leg_xy / 2) - (foot_y / 2 - 0.015)} -${0.0315 + foot_z / 2 + box_z / 2}" rpy="0 0 0" />
+		</xacro:make_fsensor>
+		<xacro:make_fsensor parent="${LRleg}foot" LR="${LRleg}" num="4">
+				<origin xyz="-${foot_x / 2 -0.015}  ${(ref * leg_xy / 2) - (foot_y / 2 - 0.015)} -${0.0315 + foot_z / 2 + box_z / 2}" rpy="0 0 0" />
+		</xacro:make_fsensor>
+		<joint name="${LRleg}foot_to_${LRleg}foot2" type="revolute">
+				<parent link="${LRleg}foot"/>
+				<child link="${LRleg}foot2"/>
+				<origin xyz="0 ${ref * leg_xy / 2} -${0.0315 + foot_z / 2 + foot_z / 10 + box_z}" rpy="0 0 0"/>
+				<axis xyz="0 0 1"/>
+				<limit lower="-0" upper="0" effort="0" velocity="0"/>
+		</joint>
+		<link name="${LRleg}foot2">
+				<visual>
+						<origin xyz="0 0 0" rpy="0 0 0"/>
+						<geometry>
+								<box size="${foot2_x} ${foot2_y} ${foot2_z}"/>
+						</geometry>
+						<xacro:gray/>
+				</visual>
+				<collision>
+						<origin xyz="0 0 0" rpy="0 0 0"/>
+						<geometry>
+								<box size="${foot2_x} ${foot2_y} ${foot2_z}"/>
+						</geometry>
+				</collision>
+				<inertial>
+						<origin xyz="0 0 0" rpy="0 0 0"/>
+						<xacro:box_inertial m="${foot2_mass}" d="${foot2_x}" w="${foot2_y}" h="${foot2_z}"/>
 				</inertial>
 		</link>
@@ -212,4 +284,5 @@
 		<xacro:gazebo_link ref="${LRleg}thigh" mu="0.8"/>
 		<xacro:gazebo_link ref="${LRleg}knee"  mu="0.8"/>
+		<xacro:gazebo_link ref="${LRleg}hizakozo" mu="0.8"/>
 		<xacro:gazebo_link ref="${LRleg}shin"  mu="0.8"/>
 		<xacro:gazebo_link ref="${LRleg}ankle" mu="0.8"/>
@@ -219,7 +292,8 @@
 		<xacro:gazebo_trans tran="${LRleg}hips_to_${LRleg}thigh_tran" joint="${LRleg}hips_to_${LRleg}thigh" motor="${LRleg}leg_motor2" />
 		<xacro:gazebo_trans tran="${LRleg}thigh_to_${LRleg}knee_tran" joint="${LRleg}thigh_to_${LRleg}knee" motor="${LRleg}leg_motor3" />
-		<xacro:gazebo_trans tran="${LRleg}knee_to_${LRleg}shin_tran"  joint="${LRleg}knee_to_${LRleg}shin"  motor="${LRleg}leg_motor4" />
-		<xacro:gazebo_trans tran="${LRleg}shin_to_${LRleg}ankle_tran" joint="${LRleg}shin_to_${LRleg}ankle" motor="${LRleg}leg_motor5" />
-		<xacro:gazebo_trans tran="${LRleg}ankle_to_${LRleg}foot_tran" joint="${LRleg}ankle_to_${LRleg}foot" motor="${LRleg}leg_motor6" />
+		<xacro:gazebo_trans tran="${LRleg}knee_to_${LRleg}shin_tran"  joint="${LRleg}knee_to_${LRleg}hizakozo"  motor="${LRleg}leg_motor4" />
+		<xacro:gazebo_trans tran="${LRleg}knee_to_${LRleg}shin_tran"  joint="${LRleg}hizakozo_to_${LRleg}shin"  motor="${LRleg}leg_motor5" />
+		<xacro:gazebo_trans tran="${LRleg}shin_to_${LRleg}ankle_tran" joint="${LRleg}shin_to_${LRleg}ankle" motor="${LRleg}leg_motor6" />
+		<xacro:gazebo_trans tran="${LRleg}ankle_to_${LRleg}foot_tran" joint="${LRleg}ankle_to_${LRleg}foot" motor="${LRleg}leg_motor7" />
 		<!-- set gazebo force sensor -->
 		<xacro:gazebo_ft-sensor LR="{LRleg}" joint="${LRleg}fsensor1_joint" num="1"/>

File: urdf/sensor/khr-force_sensor.xacro (robot description, xacro)
@@ -1,11 +1,34 @@
 <?xml version="1.0"?>
 <robot xmlns:xacro="http://ros.org/wiki/xacro">
+<xacro:include filename="$(find sotuken2017)/urdf/urdf_gazebo.xacro"/>
+	<property name="box_xy" value="0.02"/>
+	<property name="box_z" value="0.01"/>
+	<property name="box_mass" value="0.005"/>
 	<xacro:macro name="make_fsensor" params="parent LR num *joint_origin">
- 		<joint name="${LR}fsensor${num}_joint" type="fixed">
+ 		<joint name="${LR}fsensor${num}_joint" type="revolute">
    			<insert_block name="joint_origin"/>
    			<parent link="${parent}" />
    			<child link="${LR}fsensor${num}" />
+   			<axis xyz="0 0 1"/>
+			<limit lower="-0" upper="0" effort="0" velocity="0"/>
  		</joint>
 		<link name="${LR}fsensor${num}">
+			<visual>
+				<origin xyz="0 0 0" rpy="0 0 0"/>
+				<geometry>
+					<box size="${box_xy} ${box_xy} ${box_z}"/>
+				</geometry>
+				<xacro:red/>
+			</visual>
+			<collision>
+				<origin xyz="0 0 0" rpy="0 0 0"/>
+				<geometry>
+					<box size="${box_xy} ${box_xy} ${box_z}"/>
+				</geometry>
+			</collision>
+			<inertial>
+				<origin xyz="0 0 0" rpy="0 0 0"/>
+				<xacro:box_inertial m="${box_mass}" d="${box_xy}" w="${box_xy}" h="${box_z}"/>
+			</inertial>
  		</link>
  		<sensor name="${LR}fsensor${num}_sensor" update_rate="20">
@@ -13,4 +36,5 @@
    			<parent link="${parent}" />
  		</sensor>
+		<xacro:gazebo_link_red ref="${LR}fsensor${num}"/>
 	</xacro:macro>
 </robot>
