Commit message: edit khr part and add khr urdf/wrl file

File: urdf/common.xacro (robot description, xacro)
@@ -4,6 +4,21 @@
   <!-- common color -->
   <xacro:macro name="set_color">
-	  <material name="green">
-   		<color rgba="0.0 1.0 0.0 1.0"/>
+	  <material name="default">
+   		<color rgba="0.8 0.8 0.8 1.0"/>
+  	  </material>
+  </xacro:macro>
+  <xacro:macro name="silver">
+	  <material name="silver">
+   		<color rgba="${192 / 255} ${192 / 255} ${192 / 255} 1.0"/>
+  	  </material>
+  </xacro:macro>
+  <xacro:macro name="darkgray">
+	  <material name="dimgray">
+   		<color rgba="${105 / 255} ${105 / 255} ${105 / 255} 1.0"/>
+  	  </material>
+  </xacro:macro>
+  <xacro:macro name="lightgray">
+	  <material name="lightgray">
+   		<color rgba="${211 / 255} ${211 / 255} ${211 / 255} 1.0"/>
   	  </material>
   </xacro:macro>

File: urdf/khr_arm/khr-arm normal.xacro (robot description, xacro)
@@ -6,9 +6,9 @@
   <property name="arm_xy" value="0.026"/>
   <property name="shoulder_z" value="0.036"/>
-  <property name="shoulder_mass" value="0.02975"/>
+  <property name="shoulder_mass" value="0.0625"/>
   <property name="upper_arm_z" value="0.082"/>
-  <property name="upper_arm_mass" value="0.02975"/>
+  <property name="upper_arm_mass" value="0.0625"/>
   <property name="lower_arm_z" value="0.056"/>
-  <property name="lower_arm_mass" value="0.051"/>
+  <property name="lower_arm_mass" value="0.025"/>
  <xacro:macro name="make_arm" params="parent LRarm ref arm_bool">
      <joint name="${parent}_to_${LRarm}shoulder" type="revolute">
@@ -26,5 +26,5 @@
                 <box size="${arm_xy} ${arm_xy} ${shoulder_z}"/>
             </geometry>
-            <xacro:set_color/>
+            <xacro:darkgray/>
         </visual>
         <collision>
@@ -58,5 +58,5 @@
                 <box size="${arm_xy} ${arm_xy} ${upper_arm_z}"/>
             </geometry>
-            <xacro:set_color/>
+            <xacro:darkgray/>
         </visual>
         <collision>
@@ -85,5 +85,5 @@
                 <box size="${arm_xy} ${arm_xy} ${lower_arm_z}"/>
             </geometry>
-            <xacro:set_color/>
+            <xacro:darkgray/>
         </visual>
         <collision>

File: urdf/khr_body/khr-body normal.xacro (robot description, xacro)
@@ -7,9 +7,9 @@
   <property name="body_y" value="0.105"/>
   <property name="body_z" value="0.062"/>
-  <property name="body_mass" value="0.3655"/>
+  <property name="body_mass" value="0.3"/>
   <property name="body_2_x" value="0.057"/>
   <property name="body_2_y" value="0.08"/>
   <property name="body_2_z" value="0.041"/>
-  <property name="body_2_mass" value="0.3655"/>
+  <property name="body_2_mass" value="0.2"/>
   <xacro:macro name="default_origin">
 	  <origin xyz="0 0 0" rpy="0 0 0"/>
@@ -22,5 +22,5 @@
           <box size="${body_x} ${body_y} ${body_z}"/>
         </geometry>
-        <xacro:set_color/>
+        <xacro:silver/>
       </visual>
       <collision>
@@ -49,5 +49,5 @@
           <box size="${body_2_x} ${body_2_y} ${body_2_z}"/>
         </geometry>
-        <xacro:set_color/>
+        <xacro:darkgray/>
       </visual>
 	  <collision>

File: urdf/khr_head/khr-head normal.xacro (robot description, xacro)
@@ -8,5 +8,5 @@
   <property name="head_y" value="0.031"/>
   <property name="head_z" value="0.033"/>
-  <property name="head_mass" value="0.119"/>
+  <property name="head_mass" value="0.1"/>
    <xacro:macro name="make_head" params="parent">
      <joint name="${parent}_to_head" type="revolute">
@@ -24,5 +24,5 @@
         		<box size="${head_x} ${head_y} ${head_z}"/>
        		</geometry>
-       		<xacro:set_color/>
+       		<xacro:silver/>
        	</visual>
        	<collision>

File: urdf/khr_leg/khr-leg normal.xacro (robot description, xacro)
@@ -4,20 +4,20 @@
 <xacro:include filename="$(find sotuken2017)/urdf/sensor/khr-force_sensor normal.xacro"/>
 	<property name="ef" value="1.37293"/>
-  <property name="vel" value="0.14"/>
+    <property name="vel" value="0.14"/>
 	<property name="leg_xy" value="0.03"/>
 	<property name="hips_z" value="0.0039"/>
-	<property name="hips_mass" value="0.03944"/>
+	<property name="hips_mass" value="0.048"/>
 	<property name="thigh_z" value="0.026"/>
-	<property name="thigh_mass" value="0.03944"/>
+	<property name="thigh_mass" value="0.068"/>
 	<property name="knee_z" value="0.088"/>
-	<property name="knee_mass" value="0.11832"/>
+	<property name="knee_mass" value="0.118"/>
 	<property name="shin_z" value="0.047"/>
-	<property name="shin_mass" value="0.04692"/>
+	<property name="shin_mass" value="0.068"/>
 	<property name="ankle_z" value="0.02"/>
-	<property name="ankle_mass" value="0.04692"/>
+	<property name="ankle_mass" value="0.068"/>
 	<property name="foot_x" value="0.122"/>
 	<property name="foot_y" value="0.078"/>
 	<property name="foot_z" value="0.01"/>
-	<property name="foot_mass" value="0.02346"/>
+	<property name="foot_mass" value="0.03"/>
 	<property name="foot2_x" value="0.122"/>
 	<property name="foot2_y" value="0.078"/>
@@ -44,5 +44,5 @@
     							<box size="${leg_xy} ${leg_xy} ${hips_z}"/>
   						</geometry>
-  						<xacro:set_color/>
+  						<xacro:darkgray/>
   				</visual>
   				<collision>
@@ -76,5 +76,5 @@
 								<box size="${leg_xy} ${leg_xy} ${thigh_z}"/>
 						</geometry>
-						<xacro:set_color/>
+						<xacro:darkgray/>
 				</visual>
 				<collision>
@@ -103,5 +103,5 @@
 								<box size="${leg_xy} ${leg_xy} ${knee_z}"/>
 						</geometry>
-						<xacro:set_color/>
+						<xacro:darkgray/>
 				</visual>
 				<collision>
@@ -130,5 +130,5 @@
 								<box size="${leg_xy} ${leg_xy} ${shin_z}"/>
 						</geometry>
-						<xacro:set_color/>
+						<xacro:darkgray/>
 				</visual>
 				<collision>
@@ -157,5 +157,5 @@
 								<box size="${leg_xy} ${leg_xy} ${ankle_z}"/>
 						</geometry>
-						<xacro:set_color/>
+						<xacro:darkgray/>
 				</visual>
 				<collision>
@@ -184,5 +184,5 @@
 								<box size="${foot_x} ${foot_y} ${foot_z}"/>
 						</geometry>
-						<xacro:set_color/>
+						<xacro:darkgray/>
 				</visual>
 				<collision>
@@ -221,5 +221,5 @@
 								<box size="${foot2_x} ${foot2_y} ${foot2_z}"/>
 						</geometry>
-						<xacro:set_color/>
+						<xacro:darkgray/>
 				</visual>
 				<collision>

File: urdf/khr_leg/khr-leg normal_2.xacro (robot description, xacro)
@@ -4,20 +4,20 @@
 <xacro:include filename="$(find sotuken2017)/urdf/sensor/khr-force_sensor normal_2.xacro"/>
 	<property name="ef" value="1.37293"/>
-  <property name="vel" value="0.14"/>
+    <property name="vel" value="0.14"/>
 	<property name="leg_xy" value="0.03"/>
 	<property name="hips_z" value="0.0039"/>
-	<property name="hips_mass" value="0.03944"/>
+	<property name="hips_mass" value="0.048"/>
 	<property name="thigh_z" value="0.026"/>
-	<property name="thigh_mass" value="0.03944"/>
+	<property name="thigh_mass" value="0.068"/>
 	<property name="knee_z" value="0.088"/>
-	<property name="knee_mass" value="0.11832"/>
+	<property name="knee_mass" value="0.118"/>
 	<property name="shin_z" value="0.047"/>
-	<property name="shin_mass" value="0.04692"/>
+	<property name="shin_mass" value="0.068"/>
 	<property name="ankle_z" value="0.02"/>
-	<property name="ankle_mass" value="0.04692"/>
+	<property name="ankle_mass" value="0.068"/>
 	<property name="foot_x" value="0.122"/>
 	<property name="foot_y" value="0.078"/>
 	<property name="foot_z" value="0.01"/>
-	<property name="foot_mass" value="0.02346"/>
+	<property name="foot_mass" value="0.03"/>
 	<property name="foot2_x" value="0.122"/>
 	<property name="foot2_y" value="0.078"/>
@@ -44,5 +44,5 @@
     							<box size="${leg_xy} ${leg_xy} ${hips_z}"/>
   						</geometry>
-  						<xacro:set_color/>
+  						<xacro:darkgray/>
   				</visual>
   				<collision>
@@ -76,5 +76,5 @@
 								<box size="${leg_xy} ${leg_xy} ${thigh_z}"/>
 						</geometry>
-						<xacro:set_color/>
+						<xacro:darkgray/>
 				</visual>
 				<collision>
@@ -103,5 +103,5 @@
 								<box size="${leg_xy} ${leg_xy} ${knee_z}"/>
 						</geometry>
-						<xacro:set_color/>
+						<xacro:darkgray/>
 				</visual>
 				<collision>
@@ -130,5 +130,5 @@
 								<box size="${leg_xy} ${leg_xy} ${shin_z}"/>
 						</geometry>
-						<xacro:set_color/>
+						<xacro:darkgray/>
 				</visual>
 				<collision>
@@ -157,5 +157,5 @@
 								<box size="${leg_xy} ${leg_xy} ${ankle_z}"/>
 						</geometry>
-						<xacro:set_color/>
+						<xacro:darkgray/>
 				</visual>
 				<collision>
@@ -184,5 +184,5 @@
 								<box size="${foot_x} ${foot_y} ${foot_z}"/>
 						</geometry>
-						<xacro:set_color/>
+						<xacro:darkgray/>
 				</visual>
 				<collision>
@@ -223,5 +223,5 @@
 								<box size="${foot2_x} ${foot2_y} ${foot2_z}"/>
 						</geometry>
-						<xacro:set_color/>
+						<xacro:darkgray/>
 				</visual>
 				<collision>

File: urdf/sensor/khr-force_sensor normal.xacro (robot description, xacro)
@@ -16,5 +16,5 @@
 					<box size="${box_xy} ${box_xy} ${box_z}"/>
 				</geometry>
-				<xacro:set_color/>
+				<xacro:lightgray/>
 			</visual>
 			<collision>

File: urdf/sensor/khr-force_sensor normal_2.xacro (robot description, xacro)
@@ -18,5 +18,5 @@
 					<box size="${box_xy} ${box_xy} ${box_z}"/>
 				</geometry>
-				<xacro:set_color/>
+				<xacro:lightgray/>
 			</visual>
 			<collision>

Commit message: add gazebo color

File: urdf/common.xacro (robot description, xacro)
@@ -8,17 +8,17 @@
   	  </material>
   </xacro:macro>
+  <xacro:macro name="red">
+	  <material name="red">
+   		<color rgba="1.0 0.0 0.0 1.0"/>
+  	  </material>
+  </xacro:macro>
+  <xacro:macro name="black">
+	  <material name="black">
+   		<color rgba="0.3 0.3 0.3 1.0"/>
+  	  </material>
+  </xacro:macro>
   <xacro:macro name="silver">
 	  <material name="silver">
    		<color rgba="${192 / 255} ${192 / 255} ${192 / 255} 1.0"/>
-  	  </material>
-  </xacro:macro>
-  <xacro:macro name="darkgray">
-	  <material name="dimgray">
-   		<color rgba="${105 / 255} ${105 / 255} ${105 / 255} 1.0"/>
-  	  </material>
-  </xacro:macro>
-  <xacro:macro name="lightgray">
-	  <material name="lightgray">
-   		<color rgba="${211 / 255} ${211 / 255} ${211 / 255} 1.0"/>
   	  </material>
   </xacro:macro>

File: urdf/khr_arm/khr-arm normal.xacro (robot description, xacro)
@@ -2,4 +2,5 @@
 <robot xmlns:xacro="http://ros.org/wiki/xacro">
 <xacro:include filename="$(find sotuken2017)/urdf/common.xacro"/>
+<xacro:include filename="$(find sotuken2017)/urdf/urdf_gazebo.xacro"/>
   <property name="ef" value="1.37293"/>
   <property name="vel" value="0.14"/>
@@ -26,5 +27,5 @@
                 <box size="${arm_xy} ${arm_xy} ${shoulder_z}"/>
             </geometry>
-            <xacro:darkgray/>
+            <xacro:black/>
         </visual>
         <collision>
@@ -58,5 +59,5 @@
                 <box size="${arm_xy} ${arm_xy} ${upper_arm_z}"/>
             </geometry>
-            <xacro:darkgray/>
+            <xacro:black/>
         </visual>
         <collision>
@@ -85,5 +86,5 @@
                 <box size="${arm_xy} ${arm_xy} ${lower_arm_z}"/>
             </geometry>
-            <xacro:darkgray/>
+            <xacro:black/>
         </visual>
         <collision>
@@ -98,4 +99,7 @@
         </inertial>
     </link>
+	<xacro:gazebo_link_black ref="${LRarm}shoulder"/>
+	<xacro:gazebo_link_black ref="${LRarm}upper_arm"/>
+	<xacro:gazebo_link_black ref="${LRarm}lower_arm"/>
   </xacro:macro>
 </robot>

File: urdf/khr_body/khr-body normal.xacro (robot description, xacro)
@@ -2,4 +2,5 @@
 <robot xmlns:xacro="http://ros.org/wiki/xacro">
 <xacro:include filename="$(find sotuken2017)/urdf/common.xacro"/>
+<xacro:include filename="$(find sotuken2017)/urdf/urdf_gazebo.xacro"/>
   <property name="ef" value="1.37293"/>
   <property name="vel" value="0.14"/>
@@ -49,5 +50,5 @@
           <box size="${body_2_x} ${body_2_y} ${body_2_z}"/>
         </geometry>
-        <xacro:darkgray/>
+        <xacro:black/>
       </visual>
 	  <collision>
@@ -62,4 +63,6 @@
       </inertial>
     </link>
+	<xacro:gazebo_link_gray ref="base_link"/>
+	<xacro:gazebo_link_black ref="body_2"/>
   </xacro:macro>
 </robot>

File: urdf/khr_head/khr-head normal.xacro (robot description, xacro)
@@ -2,4 +2,5 @@
 <robot xmlns:xacro="http://ros.org/wiki/xacro">
 <xacro:include filename="$(find sotuken2017)/urdf/common.xacro"/>
+<xacro:include filename="$(find sotuken2017)/urdf/urdf_gazebo.xacro"/>
 <xacro:include filename="$(find sotuken2017)/urdf/khr_body/khr-body.xacro"/>
   <property name="ef" value="1.37293"/>
@@ -37,4 +38,5 @@
 	   	</inertial>
      </link>
+	 <xacro:gazebo_link_gray ref="head"/>
    </xacro:macro>
 </robot>

File: urdf/khr_leg/khr-leg normal.xacro (robot description, xacro)
@@ -2,4 +2,5 @@
 <robot xmlns:xacro="http://ros.org/wiki/xacro">
 <xacro:include filename="$(find sotuken2017)/urdf/common.xacro"/>
+<xacro:include filename="$(find sotuken2017)/urdf/urdf_gazebo.xacro"/>
 <xacro:include filename="$(find sotuken2017)/urdf/sensor/khr-force_sensor normal.xacro"/>
 	<property name="ef" value="1.37293"/>
@@ -44,5 +45,5 @@
     							<box size="${leg_xy} ${leg_xy} ${hips_z}"/>
   						</geometry>
-  						<xacro:darkgray/>
+  						<xacro:black/>
   				</visual>
   				<collision>
@@ -76,5 +77,5 @@
 								<box size="${leg_xy} ${leg_xy} ${thigh_z}"/>
 						</geometry>
-						<xacro:darkgray/>
+						<xacro:black/>
 				</visual>
 				<collision>
@@ -103,5 +104,5 @@
 								<box size="${leg_xy} ${leg_xy} ${knee_z}"/>
 						</geometry>
-						<xacro:darkgray/>
+						<xacro:black/>
 				</visual>
 				<collision>
@@ -130,5 +131,5 @@
 								<box size="${leg_xy} ${leg_xy} ${shin_z}"/>
 						</geometry>
-						<xacro:darkgray/>
+						<xacro:black/>
 				</visual>
 				<collision>
@@ -157,5 +158,5 @@
 								<box size="${leg_xy} ${leg_xy} ${ankle_z}"/>
 						</geometry>
-						<xacro:darkgray/>
+						<xacro:black/>
 				</visual>
 				<collision>
@@ -184,5 +185,5 @@
 								<box size="${foot_x} ${foot_y} ${foot_z}"/>
 						</geometry>
-						<xacro:darkgray/>
+						<xacro:black/>
 				</visual>
 				<collision>
@@ -221,5 +222,5 @@
 								<box size="${foot2_x} ${foot2_y} ${foot2_z}"/>
 						</geometry>
-						<xacro:darkgray/>
+						<xacro:black/>
 				</visual>
 				<collision>
@@ -234,4 +235,11 @@
 				</inertial>
 		</link>
+		<xacro:gazebo_link_black ref="${LRleg}hips"/>
+		<xacro:gazebo_link_black ref="${LRleg}thigh"/>
+		<xacro:gazebo_link_black ref="${LRleg}knee"/>
+		<xacro:gazebo_link_black ref="${LRleg}shin"/>
+		<xacro:gazebo_link_black ref="${LRleg}ankle"/>
+		<xacro:gazebo_link_black ref="${LRleg}foot"/>
+		<xacro:gazebo_link_gray ref="${LRleg}foot2"/>
 	</xacro:macro>
 </robot>

File: urdf/khr_leg/khr-leg normal_2.xacro (robot description, xacro)
@@ -2,4 +2,5 @@
 <robot xmlns:xacro="http://ros.org/wiki/xacro">
 <xacro:include filename="$(find sotuken2017)/urdf/common.xacro"/>
+<xacro:include filename="$(find sotuken2017)/urdf/urdf_gazebo.xacro"/>
 <xacro:include filename="$(find sotuken2017)/urdf/sensor/khr-force_sensor normal_2.xacro"/>
 	<property name="ef" value="1.37293"/>
@@ -44,5 +45,5 @@
     							<box size="${leg_xy} ${leg_xy} ${hips_z}"/>
   						</geometry>
-  						<xacro:darkgray/>
+  						<xacro:black/>
   				</visual>
   				<collision>
@@ -76,5 +77,5 @@
 								<box size="${leg_xy} ${leg_xy} ${thigh_z}"/>
 						</geometry>
-						<xacro:darkgray/>
+						<xacro:black/>
 				</visual>
 				<collision>
@@ -103,5 +104,5 @@
 								<box size="${leg_xy} ${leg_xy} ${knee_z}"/>
 						</geometry>
-						<xacro:darkgray/>
+						<xacro:black/>
 				</visual>
 				<collision>
@@ -130,5 +131,5 @@
 								<box size="${leg_xy} ${leg_xy} ${shin_z}"/>
 						</geometry>
-						<xacro:darkgray/>
+						<xacro:black/>
 				</visual>
 				<collision>
@@ -157,5 +158,5 @@
 								<box size="${leg_xy} ${leg_xy} ${ankle_z}"/>
 						</geometry>
-						<xacro:darkgray/>
+						<xacro:black/>
 				</visual>
 				<collision>
@@ -184,5 +185,5 @@
 								<box size="${foot_x} ${foot_y} ${foot_z}"/>
 						</geometry>
-						<xacro:darkgray/>
+						<xacro:black/>
 				</visual>
 				<collision>
@@ -223,5 +224,5 @@
 								<box size="${foot2_x} ${foot2_y} ${foot2_z}"/>
 						</geometry>
-						<xacro:darkgray/>
+						<xacro:silver/>
 				</visual>
 				<collision>
@@ -236,4 +237,11 @@
 				</inertial>
 		</link>
+		<xacro:gazebo_link_black ref="${LRleg}hips"/>
+		<xacro:gazebo_link_black ref="${LRleg}thigh"/>
+		<xacro:gazebo_link_black ref="${LRleg}knee"/>
+		<xacro:gazebo_link_black ref="${LRleg}shin"/>
+		<xacro:gazebo_link_black ref="${LRleg}ankle"/>
+		<xacro:gazebo_link_black ref="${LRleg}foot"/>
+		<xacro:gazebo_link_gray ref="${LRleg}foot2"/>
 	</xacro:macro>
 </robot>

File: urdf/sensor/khr-force_sensor normal.xacro (robot description, xacro)
@@ -1,4 +1,5 @@
 <?xml version="1.0"?>
 <robot xmlns:xacro="http://ros.org/wiki/xacro">
+<xacro:include filename="$(find sotuken2017)/urdf/urdf_gazebo.xacro"/>
 	<property name="box_xy" value="0.02"/>
 	<property name="box_z" value="0.01"/>
@@ -16,5 +17,5 @@
 					<box size="${box_xy} ${box_xy} ${box_z}"/>
 				</geometry>
-				<xacro:lightgray/>
+				<xacro:red/>
 			</visual>
 			<collision>
@@ -33,4 +34,5 @@
    			<parent link="${parent}" />
  		</sensor>
+		<xacro:gazebo_link_red ref="${LR}fsensor${num}"/>
 	</xacro:macro>
 </robot>

File: urdf/sensor/khr-force_sensor normal_2.xacro (robot description, xacro)
@@ -1,4 +1,5 @@
 <?xml version="1.0"?>
 <robot xmlns:xacro="http://ros.org/wiki/xacro">
+<xacro:include filename="$(find sotuken2017)/urdf/urdf_gazebo.xacro"/>
 	<property name="box_xy" value="0.02"/>
 	<property name="box_z" value="0.01"/>
@@ -18,5 +19,5 @@
 					<box size="${box_xy} ${box_xy} ${box_z}"/>
 				</geometry>
-				<xacro:lightgray/>
+				<xacro:red/>
 			</visual>
 			<collision>
@@ -35,4 +36,5 @@
    			<parent link="${parent}" />
  		</sensor>
+		<xacro:gazebo_link_red ref="${LR}fsensor${num}"/>
 	</xacro:macro>
 </robot>

File: urdf/urdf_gazebo.xacro (robot description, xacro)
@@ -1,4 +1,27 @@
 <?xml version="1.0"?>
 <robot xmlns:xacro="http://ros.org/wiki/xacro">
+  <xacro:macro name="gazebo_link" params="ref mu" >
+	<gazebo reference="${ref}">
+	  <selfCollide>false</selfCollide>
+      <mu1 value="${mu}" />
+      <mu2 value="${mu}" />
+	  <material>Gazebo/Green</material>
+    </gazebo>
+  </xacro:macro>
+  <xacro:macro name="gazebo_link_red" params="ref">
+	<gazebo reference="${ref}">
+	  <material>Gazebo/Red</material>
+    </gazebo>
+  </xacro:macro>
+  <xacro:macro name="gazebo_link_black" params="ref">
+	<gazebo reference="${ref}">
+	  <material>Gazebo/Black</material>
+    </gazebo>
+  </xacro:macro>
+  <xacro:macro name="gazebo_link_gray" params="ref">
+	<gazebo reference="${ref}">
+	  <material>Gazebo/Grey</material>
+    </gazebo>
+  </xacro:macro>
   <!-- ros_control plugin -->
   <xacro:macro name="gazebo_control" params="robot">
@@ -10,12 +33,5 @@
   	</gazebo>
   </xacro:macro>
-  <xacro:macro name="gazebo_link" params="ref mu" >
-	<gazebo reference="${ref}">
-	  <selfCollide>false</selfCollide>
-      <mu1 value="${mu}" />
-      <mu2 value="${mu}" />
-	  <material>Gazebo/Green</material>
-    </gazebo>
-  </xacro:macro>
+  <!-- gazebo transmission(type effort) -->
   <xacro:macro name="gazebo_trans" params="tran joint motor" >
   	<transmission name="${tran}">

Commit message: edit khr part

File: urdf/common.xacro (robot description, xacro)
@@ -18,7 +18,7 @@
   	  </material>
   </xacro:macro>
-  <xacro:macro name="silver">
-	  <material name="silver">
-   		<color rgba="${192 / 255} ${192 / 255} ${192 / 255} 1.0"/>
+  <xacro:macro name="gray">
+	  <material name="gray">
+   		<color rgba="0.8 0.8 0.8 1.0"/>
   	  </material>
   </xacro:macro>

File: urdf/khr_body/khr-body normal.xacro (robot description, xacro)
@@ -23,5 +23,5 @@
           <box size="${body_x} ${body_y} ${body_z}"/>
         </geometry>
-        <xacro:silver/>
+        <xacro:gray/>
       </visual>
       <collision>

File: urdf/khr_head/khr-head normal.xacro (robot description, xacro)
@@ -25,5 +25,5 @@
         		<box size="${head_x} ${head_y} ${head_z}"/>
        		</geometry>
-       		<xacro:silver/>
+       		<xacro:gray/>
        	</visual>
        	<collision>

File: urdf/khr_leg/khr-leg normal.xacro (robot description, xacro)
@@ -222,5 +222,5 @@
 								<box size="${foot2_x} ${foot2_y} ${foot2_z}"/>
 						</geometry>
-						<xacro:black/>
+						<xacro:gray/>
 				</visual>
 				<collision>
