Commit message: add urdf/wrl file and edit khr head/body

File: robot/urdf-temp/khr-3hv.urdf (robot description, URDF)
Before this commit: robot khr-3hv, 31 links, 30 joints
Links:
- link base_link: mass 0.3655 -> 0.3
- link body_2: mass 0.3655 -> 0.2

File: urdf/khr_head/khr-head normal.xacro (robot description, xacro)
@@ -3,5 +3,5 @@
 <xacro:include filename="$(find sotuken2017)/urdf/common.xacro"/>
 <xacro:include filename="$(find sotuken2017)/urdf/urdf_gazebo.xacro"/>
-<xacro:include filename="$(find sotuken2017)/urdf/khr_body/khr-body.xacro"/>
+<xacro:include filename="$(find sotuken2017)/urdf/khr_body/khr-body normal.xacro"/>
   <property name="ef" value="1.37293"/>
   <property name="vel" value="0.14"/>
