Commit message: add khr-3hv file and wrl file

File: urdf/khr_leg/khr-leg_foot3.xacro (robot description, xacro)
@@ -15,6 +15,8 @@
 	<property name="shin_z" value="0.047"/>
 	<property name="shin_mass" value="0.068"/>
+	<property name="hizakozo_xz" value="0.01"/>
+	<property name="hizakozo_mass" value="0.01"/>
 	<property name="ankle_z" value="0.02"/>
-	<property name="ankle_mass" value="0.068"/>
+	<property name="ankle_mass" value="0.058"/>
 	<property name="foot_x" value="0.122"/>
 	<property name="foot_y" value="0.078"/>
@@ -117,8 +119,35 @@
 				</inertial>
 		</link>
-		<joint name="${LRleg}knee_to_${LRleg}shin" type="revolute">
+		<joint name="${LRleg}knee_to_${LRleg}hizakozo" type="revolute">
 				<parent link="${LRleg}knee"/>
+				<child link="${LRleg}hizakozo"/>
+				<origin xyz="0 0 -0.078" rpy="0 0 0"/>
+				<axis xyz="0 1 0"/>
+				<dynamics damping="0.5"/>
+				<limit lower="-0.0" upper="${M_PI / 2}" effort="${ef}" velocity="${vel}"/>
+		</joint>
+		<link name="${LRleg}hizakozo">
+				<visual>
+						<origin xyz="${hizakozo_xz} 0 -0.016" rpy="0 0 0"/>
+						<geometry>
+								<box size="${hizakozo_xz} ${leg_xy} ${hizakozo_xz}"/>
+						</geometry>
+						<xacro:black/>
+				</visual>
+				<collision>
+						<origin xyz="${hizakozo_xz} 0 -0.0235" rpy="0 0 0"/>
+						<geometry>
+								<box size="${hizakozo_xz} ${leg_xy} ${hizakozo_xz}"/>
+						</geometry>
+				</collision>
+				<inertial>
+						<origin xyz="${hizakozo_xz} 0 -0.0235" rpy="0 0 0"/>
+						<xacro:box_inertial m="${hizakozo_mass}" d="${hizakozo_xz}" w="${leg_xy}" h="${hizakozo_xz}"/>
+				</inertial>
+		</link>
+		<joint name="${LRleg}hizakozo_to_${LRleg}shin" type="revolute">
+				<parent link="${LRleg}hizakozo"/>
 				<child link="${LRleg}shin"/>
-				<origin xyz="0 0 -0.0885" rpy="0 0 0"/>
+				<origin xyz="0 0 -0.032" rpy="0 0 0"/>
 				<axis xyz="0 1 0"/>
 				<dynamics damping="0.5"/>
@@ -127,5 +156,5 @@
 		<link name="${LRleg}shin">
 				<visual>
-						<origin xyz="0 0 -0.024" rpy="0 0 0"/>
+						<origin xyz="0 0 -0.0235" rpy="0 0 0"/>
 						<geometry>
 								<box size="${leg_xy} ${leg_xy} ${shin_z}"/>
@@ -134,5 +163,5 @@
 				</visual>
 				<collision>
-						<origin xyz="0 0 -0.024" rpy="0 0 0"/>
+						<origin xyz="0 0 -0.0235" rpy="0 0 0"/>
 						<geometry>
 								<box size="${leg_xy} ${leg_xy} ${shin_z}"/>
@@ -140,5 +169,5 @@
 				</collision>
 				<inertial>
-						<origin xyz="0 0 -0.024" rpy="0 0 0"/>
+						<origin xyz="0 0 -0.0235" rpy="0 0 0"/>
 						<xacro:box_inertial m="${shin_mass}" d="${leg_xy}" w="${leg_xy}" h="${shin_z}"/>
 				</inertial>
@@ -240,4 +269,5 @@
 		<xacro:gazebo_link_black ref="${LRleg}thigh"/>
 		<xacro:gazebo_link_black ref="${LRleg}knee"/>
+		<xacro:gazebo_link_black ref="${LRleg}hizakozo"/>
 		<xacro:gazebo_link_black ref="${LRleg}shin"/>
 		<xacro:gazebo_link_black ref="${LRleg}ankle"/>

Commit message: change khr-3hv_ver3 file

File: urdf/khr_leg/khr-leg_foot3.xacro (robot description, xacro)
@@ -136,5 +136,5 @@
 				</visual>
 				<collision>
-						<origin xyz="${hizakozo_xz} 0 -0.0235" rpy="0 0 0"/>
+						<origin xyz="${hizakozo_xz} 0 -0.016" rpy="0 0 0"/>
 						<geometry>
 								<box size="${hizakozo_xz} ${leg_xy} ${hizakozo_xz}"/>
@@ -142,5 +142,5 @@
 				</collision>
 				<inertial>
-						<origin xyz="${hizakozo_xz} 0 -0.0235" rpy="0 0 0"/>
+						<origin xyz="${hizakozo_xz} 0 -0.016" rpy="0 0 0"/>
 						<xacro:box_inertial m="${hizakozo_mass}" d="${hizakozo_xz}" w="${leg_xy}" h="${hizakozo_xz}"/>
 				</inertial>
